File: SingleCharger/Power Delivery.kicad_sch (KiCad schematic)
At the start: 46 parts, among them J3 Conn_01x02_Pin, U3 TPS54360BDDAR, U4 TPS54360BDDAR, U5 TPS54360BDDAR

Commit message: Finished with layout changes.
Parts:
- J3: footprint Connector_PinHeader_2.54mm:PinHeader_1x02_P2.54mm_Vertical -> Connector_PinHeader_2.54mm:PinHeader_1x02_P2.54mm_Horizontal
Changed lines of the file:
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@@
 			)
 		)
-		(property "Footprint" "Connector_PinHeader_2.54mm:PinHeader_1x02_P2.54mm_Vertical"
+		(property "Footprint" "Connector_PinHeader_2.54mm:PinHeader_1x02_P2.54mm_Horizontal"
 			(at 189.23 34.29 0)
 			(effects
