File: SingleCharger/SingleCharger.kicad_pcb (KiCad board)
At the start: 2 copper layers, 120 x 130 mm, 94 parts, among them J1 Bus_PCI_Express_x1, J2 Conn_01x03_Pin, J3 Conn_01x02_Pin, J4 Conn_01x02_Pin, J5 Conn_01x03_Pin, Q2 TPHR8504PL,LQ(M1W, Q5 NMOS, Q6 NMOS, Q7 NMOS, Q8 NMOS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

Commit message: Updated Silkscreen
Other:
- board text added: "V1.3"
- board text removed: "V1.2"
Changed lines of the file:
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@@
 		)
 	)
-	(gr_text "V1.2"
+	(gr_text "V1.3"
 		(at 138.938 136.398 0)
 		(layer "F.SilkS" knockout)
@@
 			)
 		)
-		(render_cache "V1.2" 0
+		(render_cache "V1.3" 0
 			(polygon
 				(pts
-					(xy 137.843762 135.496424) (xy 137.287346 137.0205) (xy 136.846793 137.0205) (xy 136.290377 135.496424)
-					(xy 136.70327 135.496424) (xy 137.072199 136.567032) (xy 137.441036 135.496424)
+					(xy 136.817117 135.434875) (xy 137.199327 136.400153) (xy 137.583551 135.434875) (xy 138.030882 135.434875)
+					(xy 137.363092 137.0205) (xy 137.03547 137.0205) (xy 136.369787 135.434875)
 				)
 			)
 			(polygon
 				(pts
-					(xy 139.160017 137.0205) (xy 138.141525 137.0205) (xy 138.141525 136.756717) (xy 138.463284 136.756717)
-					(xy 138.463284 135.947785) (xy 138.141525 135.947785) (xy 138.141525 135.701588) (xy 138.282941 135.692979)
-					(xy 138.347231 135.680616) (xy 138.39569 135.663211) (xy 138.443252 135.633336) (xy 138.475557 135.597541)
-					(xy 138.496131 135.553468) (xy 138.506332 135.496424) (xy 138.845494 135.496424) (xy 138.845494 136.756717)
-					(xy 139.160017 136.756717)
+					(xy 138.587023 135.783654) (xy 138.355481 135.783654) (xy 138.355481 135.431944) (xy 138.997351 135.431944)
+					(xy 138.997351 137.0205) (xy 138.587023 137.0205)
 				)
 			)
 			(polygon
 				(pts
-					(xy 139.931489 137.0205) (xy 139.548272 137.0205) (xy 139.548272 136.616033) (xy 139.931489 136.616033)
+					(xy 139.476556 136.821106) (xy 139.481326 136.771859) (xy 139.495515 136.725485) (xy 139.518238 136.682996)
+					(xy 139.548088 136.646625) (xy 139.584527 136.616692) (xy 139.626948 136.59396) (xy 139.673347 136.579775)
+					(xy 139.722752 136.575001) (xy 139.772158 136.579775) (xy 139.818557 136.59396) (xy 139.861038 136.616702)
+					(xy 139.897416 136.646625) (xy 139.927319 136.683006) (xy 139.94999 136.725485) (xy 139.964179 136.771859)
+					(xy 139.968949 136.821106) (xy 139.964175 136.870511) (xy 139.94999 136.91691) (xy 139.927323 136.959405)
+					(xy 139.897416 136.995862) (xy 139.861045 137.025711) (xy 139.818557 137.048435) (xy 139.772158 137.06262)
+					(xy 139.722752 137.067394) (xy 139.673347 137.06262) (xy 139.626948 137.048435) (xy 139.58452 137.025721)
+					(xy 139.548088 136.995862) (xy 139.518234 136.959415) (xy 139.495515 136.91691) (xy 139.48133 136.870511)
 				)
 			)
 			(polygon
 				(pts
-					(xy 141.505848 137.0205) (xy 140.30802 137.0205) (xy 140.30802 136.767342) (xy 140.583068 136.557507)
-					(xy 140.712969 136.449105) (xy 140.803894 136.36599) (xy 140.915824 136.247498) (xy 140.980115 136.158261)
-					(xy 141.0099 136.097533) (xy 141.026905 136.039452) (xy 141.032413 135.983047) (xy 141.024392 135.916849)
-					(xy 141.001899 135.864442) (xy 140.965277 135.82258) (xy 140.917337 135.792675) (xy 140.854383 135.773231)
-					(xy 140.772112 135.766068) (xy 140.677417 135.775191) (xy 140.573817 135.804079) (xy 140.473162 135.847446)
-					(xy 140.380743 135.90089) (xy 140.347953 135.90089) (xy 140.347953 135.562278) (xy 140.429861 135.533011)
-					(xy 140.562551 135.498897) (xy 140.704993 135.47502) (xy 140.846942 135.467115) (xy 140.992689 135.475971)
-					(xy 141.111197 135.500395) (xy 141.207156 135.537938) (xy 141.284472 135.587282) (xy 141.349652 135.652607)
-					(xy 141.396147 135.729314) (xy 141.424977 135.819674) (xy 141.435139 135.927085) (xy 141.427154 136.021299)
-					(xy 141.403259 136.112207) (xy 141.362874 136.201034) (xy 141.30968 136.28375) (xy 141.237143 136.372738)
-					(xy 141.142048 136.468846) (xy 141.047755 136.551888) (xy 140.954469 136.62675) (xy 140.820289 136.727408)
-					(xy 141.505848 136.727408)
+					(xy 140.707631 136.057053) (xy 140.735841 136.05916) (xy 140.755716 136.05916) (xy 140.805245 136.053674)
+					(xy 140.846328 136.038085) (xy 140.88083 136.012631) (xy 140.90724 135.978927) (xy 140.923234 135.939249)
+					(xy 140.928823 135.891823) (xy 140.923549 135.845703) (xy 140.908542 135.807491) (xy 140.883944 135.775411)
+					(xy 140.851631 135.750963) (xy 140.813566 135.7361) (xy 140.768081 135.730897) (xy 140.720332 135.736799)
+					(xy 140.680631 135.753696) (xy 140.647089 135.78173) (xy 140.622057 135.818) (xy 140.606638 135.861129)
+					(xy 140.601202 135.91298) (xy 140.220733 135.91298) (xy 140.244145 135.793113) (xy 140.282557 135.691147)
+					(xy 140.336828 135.600672) (xy 140.402908 135.52729) (xy 140.481927 135.468906) (xy 140.574641 135.425807)
+					(xy 140.676606 135.399924) (xy 140.792536 135.390911) (xy 140.906286 135.399422) (xy 141.005027 135.423701)
+					(xy 141.094585 135.463882) (xy 141.168426 135.516666) (xy 141.228468 135.583059) (xy 141.273114 135.66257)
+					(xy 141.300372 135.751644) (xy 141.309842 135.853721) (xy 141.304537 135.928895) (xy 141.289809 135.990452)
+					(xy 141.266886 136.040841) (xy 141.215668 136.107764) (xy 141.144246 136.166504) (xy 141.220887 136.198979)
+					(xy 141.283834 136.243929) (xy 141.33503 136.301968) (xy 141.37232 136.370068) (xy 141.395485 136.449346)
+					(xy 141.403632 136.542394) (xy 141.398325 136.619729) (xy 141.382837 136.69081) (xy 141.35747 136.756626)
+					(xy 141.302203 136.846263) (xy 141.228418 136.922497) (xy 141.138989 136.98317) (xy 141.031222 137.029567)
+					(xy 140.913328 137.057644) (xy 140.780538 137.067394) (xy 140.660576 137.059135) (xy 140.551343 137.035123)
+					(xy 140.451176 136.995953) (xy 140.360811 136.939767) (xy 140.282826 136.864923) (xy 140.216245 136.769082)
+					(xy 140.182616 136.698693) (xy 140.162847 136.630413) (xy 140.152621 136.560644) (xy 140.1492 136.489638)
+					(xy 140.559528 136.489638) (xy 140.567053 136.561161) (xy 140.587699 136.616041) (xy 140.620253 136.658165)
+					(xy 140.663912 136.689345) (xy 140.717488 136.708759) (xy 140.783743 136.715684) (xy 140.853882 136.70826)
+					(xy 140.905392 136.688247) (xy 140.942929 136.657158) (xy 140.970617 136.615644) (xy 140.98745 136.568026)
+					(xy 140.993304 136.512627) (xy 140.985884 136.446921) (xy 140.965436 136.396507) (xy 140.932853 136.357747)
+					(xy 140.890109 136.328698) (xy 140.842634 136.311316) (xy 140.788964 136.305356) (xy 140.749305 136.308471)
+					(xy 140.707631 136.315798)
 				)
 			)
