File: SingleCharger/BatteryCC.kicad_sch (KiCad schematic)
At the start: 21 parts, among them Q2 TPHR8504PL,LQ(M1W, U1 ADS1115IDGSR, U10 LM358, U11 MCP4725A0T-E/CH, U8 UCC27324DR, U9 LM393

Commit message: Started adding LEDS
Parts:
- R14, R22, R23, R25: footprint Resistor_SMD:R_1206_3216Metric_Pad1.30x1.75mm_HandSolder -> Resistor_SMD:R_1206_3216Metric

Commit message: Fixed some issues for hopeful stability in analog measuremnets.
Parts:
- added D8: B560C-13-F, COMPONENTS:SMC_L7.1-W6.2-LS8.1-RD, symbol NEW:B560C-13-F
Connections:
- net +24V: now also D8.2 (A); no longer R3.1
- new net B+: D8.1 (K), R3.1
